File: tests/BareBlinkyComplete.kicad_pcb (KiCad board)
At the start: 2 copper layers, 16 parts, among them J1 COM-15111, J2 PinHeader1.27 Shrouded 2x5, U1 LD1117S33TR, U2 STM32F103xxT6

Commit message: wip
Parts:
- moved J1 12.8 mm to (129.5, 85.5)
Changed lines of the file:
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@@
 	(footprint "Connector_USB:USB_C_Receptacle_XKB_U262-16XN-4BVC11"
 		(layer "F.Cu")
-		(at 127.66 72.875)
+		(at 129.5 85.5)
 		(descr "USB Type C, right-angle, SMT, https://datasheet.lcsc.com/szlcsc/1811141824_XKB-Enterprise-U262-161N-4BVC11_C319148.pdf")
 		(tags "USB C Type-C Receptacle SMD")

Commit message: restoring
Parts:
- turned J1 to 45 degrees
Changed lines of the file:
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@@
 	(footprint "Connector_USB:USB_C_Receptacle_XKB_U262-16XN-4BVC11"
 		(layer "F.Cu")
-		(at 129.5 85.5)
+		(at 129.5 85.5 45)
 		(descr "USB Type C, right-angle, SMT, https://datasheet.lcsc.com/szlcsc/1811141824_XKB-Enterprise-U262-161N-4BVC11_C319148.pdf")
 		(tags "USB C Type-C Receptacle SMD")
 		(property "Reference" "J1"
-			(at 0 -5.715 0)
+			(at 0 -5.715 45)
 			(layer "F.SilkS")
 			(effects
@@
 		)
 		(property "Value" "COM-15111"
-			(at 0 4.935 0)
+			(at 0 4.935 45)
 			(layer "F.Fab")
 			(effects
@@
 		)
 		(property "Footprint" ""
-			(at 0 0 0)
+			(at 0 0 45)
 			(unlocked yes)
 			(layer "F.Fab")
@@
 		)
 		(property "Datasheet" ""
-			(at 0 0 0)
+			(at 0 0 45)
 			(unlocked yes)
 			(layer "F.Fab")
@@
 		)
 		(property "Description" ""
-			(at 0 0 0)
+			(at 0 0 45)
 			(unlocked yes)
 			(layer "F.Fab")
@@
 		(attr smd)
 		(fp_line
-			(start -4.58 -1.85)
-			(end -4.58 0.07)
+			(start -4.580001 -1.85)
+			(end -4.580001 0.07)
 			(stroke
 				(width 0.12)
@@
 		)
 		(fp_line
-			(start 4.58 0.07)
-			(end 4.58 -1.85)
+			(start 4.580001 0.07)
+			(end 4.580001 -1.85)
 			(stroke
 				(width 0.12)
@@
 		)
 		(fp_text user "${REFERENCE}"
-			(at 0 0 0)
+			(at 0 0 45)
 			(layer "F.Fab")
 			(effects
@@
 		)
 		(pad "" np_thru_hole circle
-			(at -2.89 -2.605)
+			(at -2.89 -2.605 45)
 			(size 0.65 0.65)
 			(drill 0.65)
@@
 		)
 		(pad "" np_thru_hole circle
-			(at 2.89 -2.605)
+			(at 2.89 -2.605 45)
 			(size 0.65 0.65)
 			(drill 0.65)
@@
 		)
 		(pad "A1" smd rect
-			(at -3.35 -3.67)
+			(at -3.35 -3.67 45)
 			(size 0.3 1.15)
 			(layers "F.Cu" "F.Paste" "F.Mask")
@@
 		)
 		(pad "A4" smd rect
-			(at -2.55 -3.67)
+			(at -2.55 -3.67 45)
 			(size 0.3 1.15)
 			(layers "F.Cu" "F.Paste" "F.Mask")
@@
 		)
 		(pad "A5" smd rect
-			(at -1.25 -3.67)
+			(at -1.25 -3.669999 45)
 			(size 0.3 1.15)
 			(layers "F.Cu" "F.Paste" "F.Mask")
@@
 		)
 		(pad "A6" smd rect
-			(at -0.25 -3.67)
+			(at -0.25 -3.67 45)
 			(size 0.3 1.15)
 			(layers "F.Cu" "F.Paste" "F.Mask")
@@
 		)
 		(pad "A7" smd rect
-			(at 0.25 -3.67)
+			(at 0.25 -3.67 45)
 			(size 0.3 1.15)
 			(layers "F.Cu" "F.Paste" "F.Mask")
@@
 		)
 		(pad "A8" smd rect
-			(at 1.25 -3.67)
+			(at 1.25 -3.669999 45)
 			(size 0.3 1.15)
 			(layers "F.Cu" "F.Paste" "F.Mask")
 		)
 		(pad "A9" smd rect
-			(at 2.55 -3.67)
+			(at 2.55 -3.67 45)
 			(size 0.3 1.15)
 			(layers "F.Cu" "F.Paste" "F.Mask")
@@
 		)
 		(pad "A12" smd rect
-			(at 3.35 -3.67)
+			(at 3.35 -3.67 45)
 			(size 0.3 1.15)
 			(layers "F.Cu" "F.Paste" "F.Mask")
@@
 		)
 		(pad "B1" smd rect
-			(at 3.05 -3.67)
+			(at 3.05 -3.67 45)
 			(size 0.3 1.15)
 			(layers "F.Cu" "F.Paste" "F.Mask")
@@
 		)
 		(pad "B4" smd rect
-			(at 2.25 -3.67)
+			(at 2.25 -3.67 45)
 			(size 0.3 1.15)
 			(layers "F.Cu" "F.Paste" "F.Mask")
@@
 		)
 		(pad "B5" smd rect
-			(at 1.75 -3.67)
+			(at 1.75 -3.67 45)
 			(size 0.3 1.15)
 			(layers "F.Cu" "F.Paste" "F.Mask")
@@
 		)
 		(pad "B6" smd rect
-			(at 0.75 -3.67)
+			(at 0.75 -3.67 45)
 			(size 0.3 1.15)
 			(layers "F.Cu" "F.Paste" "F.Mask")
@@
 		)
 		(pad "B7" smd rect
-			(at -0.75 -3.67)
+			(at -0.75 -3.67 45)
 			(size 0.3 1.15)
 			(layers "F.Cu" "F.Paste" "F.Mask")
@@
 		)
 		(pad "B8" smd rect
-			(at -1.75 -3.67)
+			(at -1.75 -3.67 45)
 			(size 0.3 1.15)
 			(layers "F.Cu" "F.Paste" "F.Mask")
 		)
 		(pad "B9" smd rect
-			(at -2.25 -3.67)
+			(at -2.25 -3.67 45)
 			(size 0.3 1.15)
 			(layers "F.Cu" "F.Paste" "F.Mask")
@@
 		)
 		(pad "B12" smd rect
-			(at -3.05 -3.67)
+			(at -3.05 -3.67 45)
 			(size 0.3 1.15)
 			(layers "F.Cu" "F.Paste" "F.Mask")
@@
 		)
 		(pad "S1" thru_hole oval
-			(at -4.32 -3.105)
+			(at -4.32 -3.105 45)
 			(size 1 2.1)
 			(drill oval 0.6 1.7)
@@
 		)
 		(pad "S1" thru_hole oval
-			(at -4.32 1.075)
+			(at -4.32 1.075 45)
 			(size 1 1.6)
 			(drill oval 0.6 1.2)
@@
 		)
 		(pad "S1" thru_hole oval
-			(at 4.32 -3.105)
+			(at 4.32 -3.105 45)
 			(size 1 2.1)
 			(drill oval 0.6 1.7)
@@
 		)
 		(pad "S1" thru_hole oval
-			(at 4.32 1.075)
+			(at 4.32 1.075 45)
 			(size 1 1.6)
 			(drill oval 0.6 1.2)
