File: tests/UsbSublayout.kicad_pcb (KiCad board)
At the start: 2 copper layers, 3 parts, among them J1 COM-15111

Commit message: support zones
Routing:
- added copper zone on F.Cu, net usb.pwr
Changed lines of the file:
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@@
 		(net 6)
 	)
+	(zone
+		(net 4)
+		(net_name "usb.pwr")
+		(layer "F.Cu")
+		(hatch edge 0.5)
+		(connect_pads
+			(clearance 0.5)
+		)
+		(min_thickness 0.25)
+		(filled_areas_thickness no)
+		(fill
+			(thermal_gap 0.5)
+			(thermal_bridge_width 0.5)
+		)
+		(polygon
+			(pts
+				(xy 142 45) (xy 139.5 45) (xy 139.5 51) (xy 142 51)
+			)
+		)
+	)
 )
