File: sublayout/tests/UsbSublayout.kicad_pcb (KiCad board)
At the start: 2 copper layers, 3 parts, among them J1 COM-15111

Commit message: replicate w/ groups working kinda
Routing:
- net usb.gnd: track 0.00 -> 3.01 mm
- net usb.usb.dm: track 3.12 -> 2.52 mm
- net gnd: vias 0 -> 2
Other:
- board outline added: 1 x 12 mm

Commit message: replicate track netcodes and store errors
Routing:
- net usb.gnd: vias 0 -> 2
- net gnd: vias 2 -> 0
Changed lines of the file:
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@@
 	)
 	(net 0 "")
-	(net 1 "gnd")
-	(net 2 "usb.gnd")
-	(net 3 "usb.conn.cc.cc1")
-	(net 4 "usb.conn.cc.cc2")
-	(net 5 "usb.pwr")
-	(net 6 "usb.usb.dp")
-	(net 7 "usb.usb.dm")
+	(net 1 "usb.gnd")
+	(net 2 "usb.conn.cc.cc1")
+	(net 3 "usb.conn.cc.cc2")
+	(net 4 "usb.pwr")
+	(net 5 "usb.usb.dp")
+	(net 6 "usb.usb.dm")
 	(footprint "Resistor_SMD:R_0603_1608Metric"
 		(layer "F.Cu")
@@
 			(layers "F.Cu" "F.Paste" "F.Mask")
 			(roundrect_rratio 0.25)
-			(net 2 "usb.gnd")
+			(net 1 "usb.gnd")
 		)
 		(pad "2" smd roundrect
@@
 			(layers "F.Cu" "F.Paste" "F.Mask")
 			(roundrect_rratio 0.25)
-			(net 3 "usb.conn.cc.cc1")
+			(net 2 "usb.conn.cc.cc1")
 		)
 		(model "${KICAD8_3DMODEL_DIR}/Resistor_SMD.3dshapes/R_0603_1608Metric.wrl"
@@
 			(layers "F.Cu" "F.Paste" "F.Mask")
 			(roundrect_rratio 0.25)
-			(net 2 "usb.gnd")
+			(net 1 "usb.gnd")
 		)
 		(pad "2" smd roundrect
@@
 			(layers "F.Cu" "F.Paste" "F.Mask")
 			(roundrect_rratio 0.25)
-			(net 4 "usb.conn.cc.cc2")
+			(net 3 "usb.conn.cc.cc2")
 		)
 		(model "${KICAD8_3DMODEL_DIR}/Resistor_SMD.3dshapes/R_0603_1608Metric.wrl"
@@
 			(size 0.3 1.15)
 			(layers "F.Cu" "F.Paste" "F.Mask")
-			(net 2 "usb.gnd")
+			(net 1 "usb.gnd")
 		)
 		(pad "A4" smd rect
@@
 			(size 0.3 1.15)
 			(layers "F.Cu" "F.Paste" "F.Mask")
-			(net 5 "usb.pwr")
+			(net 4 "usb.pwr")
 		)
 		(pad "A5" smd rect
@@
 			(size 0.3 1.15)
 			(layers "F.Cu" "F.Paste" "F.Mask")
-			(net 3 "usb.conn.cc.cc1")
+			(net 2 "usb.conn.cc.cc1")
 		)
 		(pad "A6" smd rect
@@
 			(size 0.3 1.15)
 			(layers "F.Cu" "F.Paste" "F.Mask")
-			(net 6 "usb.usb.dp")
+			(net 5 "usb.usb.dp")
 		)
 		(pad "A7" smd rect
@@
 			(size 0.3 1.15)
 			(layers "F.Cu" "F.Paste" "F.Mask")
-			(net 7 "usb.usb.dm")
+			(net 6 "usb.usb.dm")
 		)
 		(pad "A8" smd rect
@@
 			(size 0.3 1.15)
 			(layers "F.Cu" "F.Paste" "F.Mask")
-			(net 5 "usb.pwr")
+			(net 4 "usb.pwr")
 		)
 		(pad "A12" smd rect
@@
 			(size 0.3 1.15)
 			(layers "F.Cu" "F.Paste" "F.Mask")
-			(net 2 "usb.gnd")
+			(net 1 "usb.gnd")
 		)
 		(pad "B1" smd rect
@@
 			(size 0.3 1.15)
 			(layers "F.Cu" "F.Paste" "F.Mask")
-			(net 2 "usb.gnd")
+			(net 1 "usb.gnd")
 		)
 		(pad "B4" smd rect
@@
 			(size 0.3 1.15)
 			(layers "F.Cu" "F.Paste" "F.Mask")
-			(net 5 "usb.pwr")
+			(net 4 "usb.pwr")
 		)
 		(pad "B5" smd rect
@@
 			(size 0.3 1.15)
 			(layers "F.Cu" "F.Paste" "F.Mask")
-			(net 4 "usb.conn.cc.cc2")
+			(net 3 "usb.conn.cc.cc2")
 		)
 		(pad "B6" smd rect
@@
 			(size 0.3 1.15)
 			(layers "F.Cu" "F.Paste" "F.Mask")
-			(net 6 "usb.usb.dp")
+			(net 5 "usb.usb.dp")
 		)
 		(pad "B7" smd rect
@@
 			(size 0.3 1.15)
 			(layers "F.Cu" "F.Paste" "F.Mask")
-			(net 7 "usb.usb.dm")
+			(net 6 "usb.usb.dm")
 		)
 		(pad "B8" smd rect
@@
 			(size 0.3 1.15)
 			(layers "F.Cu" "F.Paste" "F.Mask")
-			(net 5 "usb.pwr")
+			(net 4 "usb.pwr")
 		)
 		(pad "B12" smd rect
@@
 			(size 0.3 1.15)
 			(layers "F.Cu" "F.Paste" "F.Mask")
-			(net 2 "usb.gnd")
+			(net 1 "usb.gnd")
 		)
 		(pad "S1" thru_hole oval
@@
 			(layers "*.Cu" "*.Mask")
 			(remove_unused_layers no)
-			(net 2 "usb.gnd")
+			(net 1 "usb.gnd")
 		)
 		(pad "S1" thru_hole oval
@@
 			(layers "*.Cu" "*.Mask")
 			(remove_unused_layers no)
-			(net 2 "usb.gnd")
+			(net 1 "usb.gnd")
 		)
 		(pad "S1" thru_hole oval
@@
 			(layers "*.Cu" "*.Mask")
 			(remove_unused_layers no)
-			(net 2 "usb.gnd")
+			(net 1 "usb.gnd")
 		)
 		(pad "S1" thru_hole oval
@@
 			(layers "*.Cu" "*.Mask")
 			(remove_unused_layers no)
-			(net 2 "usb.gnd")
+			(net 1 "usb.gnd")
 		)
 		(model "${KICAD6_3DMODEL_DIR}/Connector_USB.3dshapes/USB_C_Receptacle_XKB_U262-16XN-4BVC11.wrl"
@@
 		(layer "Edge.Cuts")
 	)
+	(segment
+		(start 141.345 44.4475)
+		(end 141.345 44.245)
+		(width 0.5)
+		(layer "F.Cu")
+		(net 1)
+	)
+	(segment
+		(start 141.345 51.35)
+		(end 141.345 51.5525)
+		(width 0.5)
+		(layer "F.Cu")
+		(net 1)
+	)
+	(segment
+		(start 141.345 44.245)
+		(end 140.78 43.68)
+		(width 0.5)
+		(layer "F.Cu")
+		(net 1)
+	)
+	(segment
+		(start 141.345 44.95)
+		(end 141.345 44.65)
+		(width 0.2)
+		(layer "F.Cu")
+		(net 1)
+	)
+	(segment
+		(start 141.345 51.5525)
+		(end 141.345 51.755)
+		(width 0.5)
+		(layer "F.Cu")
+		(net 1)
+	)
+	(segment
+		(start 141.345 44.65)
+		(end 141.345 44.4475)
+		(width 0.5)
+		(layer "F.Cu")
+		(net 1)
+	)
+	(segment
+		(start 141.345 51.755)
+		(end 140.78 52.32)
+		(width 0.5)
+		(layer "F.Cu")
+		(net 1)
+	)
+	(segment
+		(start 141.345 51.05)
+		(end 141.345 51.35)
+		(width 0.2)
+		(layer "F.Cu")
+		(net 1)
+	)
 	(via
 		(at 145 52)
@@
 		(drill 0.3)
 		(layers "F.Cu" "B.Cu")
+		(free yes)
 		(net 1)
 	)
@@
 		(drill 0.3)
 		(layers "F.Cu" "B.Cu")
+		(free yes)
 		(net 1)
-	)
-	(segment
-		(start 141.345 44.4475)
-		(end 141.345 44.245)
-		(width 0.5)
-		(layer "F.Cu")
-		(net 2)
-	)
-	(segment
-		(start 141.345 51.35)
-		(end 141.345 51.5525)
-		(width 0.5)
-		(layer "F.Cu")
-		(net 2)
-	)
-	(segment
-		(start 141.345 44.245)
-		(end 140.78 43.68)
-		(width 0.5)
-		(layer "F.Cu")
-		(net 2)
-	)
-	(segment
-		(start 141.345 44.95)
-		(end 141.345 44.65)
-		(width 0.2)
-		(layer "F.Cu")
-		(net 2)
-	)
-	(segment
-		(start 141.345 51.5525)
-		(end 141.345 51.755)
-		(width 0.5)
-		(layer "F.Cu")
-		(net 2)
-	)
-	(segment
-		(start 141.345 44.65)
-		(end 141.345 44.4475)
-		(width 0.5)
-		(layer "F.Cu")
-		(net 2)
-	)
-	(segment
-		(start 141.345 51.755)
-		(end 140.78 52.32)
-		(width 0.5)
-		(layer "F.Cu")
-		(net 2)
-	)
-	(segment
-		(start 141.345 51.05)
-		(end 141.345 51.35)
-		(width 0.2)
-		(layer "F.Cu")
-		(net 2)
 	)
 	(segment
@@
 		(width 0.2)
 		(layer "F.Cu")
-		(net 3)
+		(net 2)
 	)
 	(segment
@@
 		(width 0.2)
 		(layer "F.Cu")
-		(net 3)
+		(net 2)
 	)
 	(segment
@@
 		(width 0.2)
 		(layer "F.Cu")
-		(net 3)
+		(net 2)
 	)
 	(segment
@@
 		(width 0.2)
 		(layer "F.Cu")
-		(net 4)
+		(net 3)
 	)
 	(segment
@@
 		(width 0.2)
 		(layer "F.Cu")
-		(net 4)
+		(net 3)
 	)
 	(segment
@@
 		(width 0.2)
 		(layer "F.Cu")
-		(net 4)
+		(net 3)
 	)
 	(segment
@@
 		(width 0.2)
 		(layer "F.Cu")
-		(net 4)
+		(net 3)
 	)
 	(segment
@@
 		(width 0.2)
 		(layer "F.Cu")
-		(net 4)
+		(net 3)
 	)
 	(segment
@@
 		(width 0.16)
 		(layer "F.Cu")
-		(net 6)
+		(net 5)
 	)
 	(segment
@@
 		(width 0.16)
 		(layer "F.Cu")
-		(net 6)
+		(net 5)
 	)
 	(segment
@@
 		(width 0.16)
 		(layer "F.Cu")
-		(net 6)
+		(net 5)
 	)
 	(segment
@@
 		(width 0.16)
 		(layer "F.Cu")
-		(net 6)
+		(net 5)
 	)
 	(segment
@@
 		(width 0.16)
 		(layer "F.Cu")
-		(net 6)
+		(net 5)
 	)
 	(segment
@@
 		(width 0.16)
 		(layer "F.Cu")
-		(net 6)
+		(net 5)
 	)
 	(segment
@@
 		(width 0.16)
 		(layer "F.Cu")
-		(net 7)
+		(net 6)
 	)
 	(segment
@@
 		(width 0.16)
 		(layer "F.Cu")
-		(net 7)
+		(net 6)
 	)
 	(segment
@@
 		(width 0.16)
 		(layer "F.Cu")
-		(net 7)
+		(net 6)
 	)
 	(segment
@@
 		(width 0.15)
 		(layer "F.Cu")
-		(net 7)
+		(net 6)
 	)
 	(segment
@@
 		(width 0.15)
 		(layer "F.Cu")
-		(net 7)
+		(net 6)
 	)
 	(segment
@@
 		(width 0.16)
 		(layer "F.Cu")
-		(net 7)
+		(net 6)
 	)
 	(segment
@@
 		(width 0.16)
 		(layer "F.Cu")
-		(net 7)
+		(net 6)
 	)
 	(zone
-		(net 5)
+		(net 4)
 		(net_name "usb.pwr")
 		(layer "F.Cu")
